Commit message: Completed Assignment 4

File: body.urdf (robot description, URDF)
Before this commit: robot robot, 3 links, 2 joints
Joints:
- removed joint BackLeg_FrontLeg
- added joint Torso_FrontLeg: type revolute, parent Torso, child FrontLeg, origin xyz=0 1 0 rpy=0 0 0, axis 0 1 0, limit lower=-3.14159 upper=3.14159 effort=0.0 velocity=0.0
- joint Torso_BackLeg: child BackLeg -> Torso; parent Torso -> BackLeg

Commit message: Completed motors up to step 15

File: body.urdf (robot description, URDF)
Before this commit: robot robot, 3 links, 2 joints
Joints:
- removed joint Torso_FrontLeg
- added joint BackLeg_FrontLeg: type revolute, parent BackLeg, child FrontLeg, origin xyz=1 0 0 rpy=0 0 0, axis 0 1 0, limit lower=-3.14159 upper=3.14159 effort=0.0 velocity=0.0
- joint Torso_BackLeg: child Torso -> BackLeg; origin xyz=0 0.5 1 rpy=0 0 0 -> xyz=0.5 0 1 rpy=0 0 0; parent BackLeg -> Torso
